File: kicad/timer.sch (KiCad schematic (older format))
At the start: 26 parts, among them IC1 ATMEGA328P-A, P1 BATTERY, P2 ICSP, Q1 NMOS, Q2 PMOS, SW1 SPST, U1 TOUCH_PAD_13, U2 MTCH6102_SSOP, U3 MCP1755ST-3302E/DB

Commit message: APA_102C
Parts:
- added U4: APA_102C, touch_timer:APA_102C, symbol APA_102C
Connections:
- net GND: now also U4.3 (GND), U4.5 (CO), U4.6 (DO)
- net POWER: now also U4.4 (VCC)
- net DI: now reaches IC1.10 ((PCINT22/OC0A/AIN0)PD6)
- net DI: now also U4.1 (DI)
- net CI: now reaches IC1.11 ((PCINT23/AIN1)PD7)
- net CI: now also U4.2 (CI)
Changed lines of the file:
@@
 Text Label 4150 4700 0    60   ~ 0
 INT
-Wire Wire Line
-	8450 4750 8100 4750
-Wire Wire Line
-	8450 4850 8100 4850
-Wire Wire Line
-	8450 5300 8100 5300
-Wire Wire Line
-	4100 4500 4450 4500
-Wire Wire Line
-	4100 4600 4650 4600
-Wire Wire Line
-	4100 4700 4850 4700
-Wire Wire Line
-	2250 4600 3000 4600
-Wire Wire Line
-	2250 4700 3000 4700
-Wire Wire Line
-	2250 4800 3000 4800
-Wire Wire Line
-	2250 4900 3000 4900
-Wire Wire Line
-	2250 5000 3000 5000
-Wire Wire Line
-	2250 5100 3000 5100
-Wire Wire Line
-	2250 5200 3000 5200
-Wire Wire Line
-	2250 5300 3000 5300
-Wire Wire Line
-	2250 5400 3000 5400
-Wire Wire Line
-	2250 5500 3000 5500
-Wire Wire Line
-	2250 5600 3000 5600
-Wire Wire Line
-	2250 5700 3000 5700
-Wire Wire Line
-	2250 5800 3000 5800
 Text Label 2750 4600 0    60   ~ 0
 RX0
@@
 	1    0    0    -1
 $EndComp
-Wire Wire Line
-	4100 4800 5050 4800
-Wire Wire Line
-	4450 3400 4450 4200
-Wire Wire Line
-	2550 3400 5050 3400
-Wire Wire Line
-	4650 4300 4650 3400
-Connection ~ 4650 3400
-Wire Wire Line
-	5050 3400 5050 4500
 Text Label 4150 4800 0    60   ~ 0
 SYNC
@@
 	1    0    0    -1
 $EndComp
-Wire Wire Line
-	3000 4500 2550 4500
-Wire Wire Line
-	2550 4200 2550 3400
-Connection ~ 4450 3400
-Wire Wire Line
-	3550 3400 3550 4200
-Connection ~ 3550 3400
 $Comp
 L C C1
@@
 	1    0    0    -1
 $EndComp
-Wire Wire Line
-	3300 3750 3800 3750
-Connection ~ 3550 3750
 $Comp
 L GND #PWR01
@@
 	1    0    0    -1
 $EndComp
-Wire Wire Line
-	3000 5900 3000 6350
-Wire Wire Line
-	3000 6350 3200 6350
-Connection ~ 3000 6000
-Wire Wire Line
-	3200 6300 3750 6300
-Wire Wire Line
-	3200 6350 3200 6300
-Connection ~ 3650 6300
 $Comp
 L R R6
@@
 Text Label 1750 2100 0    60   ~ 0
 NBASE
-Wire Wire Line
-	2300 1650 2300 1900
-Connection ~ 2300 1700
-Wire Wire Line
-	2950 2250 3450 2250
-Connection ~ 3100 2250
-Wire Wire Line
-	4050 2250 4900 2250
-Wire Wire Line
-	3750 2450 3750 2800
-Wire Wire Line
-	3100 2550 3100 2700
-Wire Wire Line
-	3100 2700 4400 2700
-Connection ~ 3750 2700
-Wire Wire Line
-	4400 2700 4400 2550
-Connection ~ 4400 2250
-Wire Wire Line
-	1400 2100 900  2100
-Wire Wire Line
-	1700 2100 2000 2100
-Wire Wire Line
-	2300 2300 2300 2750
-Wire Wire Line
-	1900 2600 2300 2600
-Connection ~ 2300 2600
-Wire Wire Line
-	1900 2300 1900 2100
-Connection ~ 1900 2100
-Wire Wire Line
-	5950 7300 6100 7300
-Wire Wire Line
-	5450 7200 5150 7200
-Wire Wire Line
-	5150 7300 5450 7300
-Wire Wire Line
-	5150 7400 5450 7400
 $Comp
 L D_Schottky D1
@@
 	1    0    0    -1
 $EndComp
-Wire Wire Line
-	4350 7200 4550 7200
-Wire Wire Line
-	4050 7200 3800 7200
 $Comp
 L GND #PWR09
@@
 	1    0    0    -1
 $EndComp
-Wire Wire Line
-	3600 7200 3400 7200
-Wire Wire Line
-	3400 7200 3400 7350
 $Comp
 L MCP1755ST-3302E/DB U3
@@
 	1    0    0    -1
 $EndComp
-Wire Wire Line
-	3700 2450 3800 2450
-Connection ~ 3750 2450
 $Comp
 L VCC #PWR010
@@
 	1    0    0    1
 $EndComp
-Wire Wire Line
-	10350 3600 10750 3600
-Wire Wire Line
-	10350 3500 10550 3500
-Wire Wire Line
-	10550 3500 10550 3600
-Connection ~ 10550 3600
-Wire Wire Line
-	10350 5600 10350 5800
-Connection ~ 10350 5700
-Wire Wire Line
-	10350 5800 10550 5800
-Wire Wire Line
-	10550 5800 10550 5950
-Wire Wire Line
-	7800 4950 8450 4950
 $Comp
 L GND #PWR012
@@
 Text Label 8100 4000 0    60   ~ 0
 SCK
-Wire Wire Line
-	8100 4000 8450 4000
 Text Label 4550 7200 0    60   ~ 0
 SCK
 Text Label 6100 7200 0    60   ~ 0
 SWITCHED_POWER
-Wire Wire Line
-	5950 7200 6100 7200
-Wire Wire Line
-	2300 1700 2650 1700
-Wire Wire Line
-	2950 1900 2950 2250
-Wire Wire Line
-	2950 1500 2950 1200
-Wire Wire Line
-	2950 1200 2300 1200
-Wire Wire Line
-	2300 1200 2300 1350
 Text Label 7900 3600 0    60   ~ 0
 NBASE_ON
-Wire Wire Line
-	7900 3600 8450 3600
 Text Label 3750 3400 0    60   ~ 0
 3V3
@@
 Text Label 8100 3900 0    60   ~ 0
 MISO
-Wire Wire Line
-	8100 3900 8450 3900
 Text Label 8100 3800 0    60   ~ 0
 MOSI
-Wire Wire Line
-	8100 3800 8450 3800
 $Comp
 L SPST SW1
@@
 	1    0    0    -1
 $EndComp
+$Comp
+L APA_102C U4
+U 1 1 5706357A
+P 7300 2150
+F 0 "U4" H 7300 1650 60  0000 C CNN
+F 1 "APA_102C" H 7300 2250 60  0000 C CNN
+F 2 "touch_timer:APA_102C" H 7300 2150 60  0001 C CNN
+F 3 "" H 7300 2150 60  0000 C CNN
+	1    7300 2150
+	1    0    0    -1
+$EndComp
+Text Label 6400 2250 0    60   ~ 0
+POWER
+$Comp
+L GND #PWR013
+U 1 1 570638A5
+P 7850 2450
+F 0 "#PWR013" H 7850 2200 50  0001 C CNN
+F 1 "GND" H 7850 2300 50  0000 C CNN
+F 2 "" H 7850 2450 50  0000 C CNN
+F 3 "" H 7850 2450 50  0000 C CNN
+	1    7850 2450
+	1    0    0    -1
+$EndComp
+Wire Wire Line
+	8450 4750 8100 4750
+Wire Wire Line
+	8450 4850 8100 4850
+Wire Wire Line
+	8450 5300 8100 5300
+Wire Wire Line
+	4100 4500 4450 4500
+Wire Wire Line
+	4100 4600 4650 4600
+Wire Wire Line
+	4100 4700 4850 4700
+Wire Wire Line
+	2250 4600 3000 4600
+Wire Wire Line
+	2250 4700 3000 4700
+Wire Wire Line
+	2250 4800 3000 4800
+Wire Wire Line
+	2250 4900 3000 4900
+Wire Wire Line
+	2250 5000 3000 5000
+Wire Wire Line
+	2250 5100 3000 5100
+Wire Wire Line
+	2250 5200 3000 5200
+Wire Wire Line
+	2250 5300 3000 5300
+Wire Wire Line
+	2250 5400 3000 5400
+Wire Wire Line
+	2250 5500 3000 5500
+Wire Wire Line
+	2250 5600 3000 5600
+Wire Wire Line
+	2250 5700 3000 5700
+Wire Wire Line
+	2250 5800 3000 5800
+Wire Wire Line
+	4100 4800 5050 4800
+Wire Wire Line
+	4450 3400 4450 4200
+Wire Wire Line
+	2550 3400 5050 3400
+Wire Wire Line
+	4650 4300 4650 3400
+Connection ~ 4650 3400
+Wire Wire Line
+	5050 3400 5050 4500
+Wire Wire Line
+	3000 4500 2550 4500
+Wire Wire Line
+	2550 4200 2550 3400
+Connection ~ 4450 3400
+Wire Wire Line
+	3550 3400 3550 4200
+Connection ~ 3550 3400
+Wire Wire Line
+	3300 3750 3800 3750
+Connection ~ 3550 3750
+Wire Wire Line
+	3000 5900 3000 6350
+Wire Wire Line
+	3000 6350 3200 6350
+Connection ~ 3000 6000
+Wire Wire Line
+	3200 6300 3750 6300
+Wire Wire Line
+	3200 6350 3200 6300
+Connection ~ 3650 6300
+Wire Wire Line
+	2300 1650 2300 1900
+Connection ~ 2300 1700
+Wire Wire Line
+	2950 2250 3450 2250
+Connection ~ 3100 2250
+Wire Wire Line
+	4050 2250 4900 2250
+Wire Wire Line
+	3750 2450 3750 2800
+Wire Wire Line
+	3100 2550 3100 2700
+Wire Wire Line
+	3100 2700 4400 2700
+Connection ~ 3750 2700
+Wire Wire Line
+	4400 2700 4400 2550
+Connection ~ 4400 2250
+Wire Wire Line
+	1400 2100 900  2100
+Wire Wire Line
+	1700 2100 2000 2100
+Wire Wire Line
+	2300 2300 2300 2750
+Wire Wire Line
+	1900 2600 2300 2600
+Connection ~ 2300 2600
+Wire Wire Line
+	1900 2300 1900 2100
+Connection ~ 1900 2100
+Wire Wire Line
+	5950 7300 6100 7300
+Wire Wire Line
+	5450 7200 5150 7200
+Wire Wire Line
+	5150 7300 5450 7300
+Wire Wire Line
+	5150 7400 5450 7400
+Wire Wire Line
+	4350 7200 4550 7200
+Wire Wire Line
+	4050 7200 3800 7200
+Wire Wire Line
+	3600 7200 3400 7200
+Wire Wire Line
+	3400 7200 3400 7350
+Wire Wire Line
+	3700 2450 3800 2450
+Connection ~ 3750 2450
+Wire Wire Line
+	10350 3600 10750 3600
+Wire Wire Line
+	10350 3500 10550 3500
+Wire Wire Line
+	10550 3500 10550 3600
+Connection ~ 10550 3600
+Wire Wire Line
+	10350 5600 10350 5800
+Connection ~ 10350 5700
+Wire Wire Line
+	10350 5800 10550 5800
+Wire Wire Line
+	10550 5800 10550 5950
+Wire Wire Line
+	7800 4950 8450 4950
+Wire Wire Line
+	8100 4000 8450 4000
+Wire Wire Line
+	5950 7200 6100 7200
+Wire Wire Line
+	2300 1700 2650 1700
+Wire Wire Line
+	2950 1900 2950 2250
+Wire Wire Line
+	2950 1500 2950 1200
+Wire Wire Line
+	2950 1200 2300 1200
+Wire Wire Line
+	2300 1200 2300 1350
+Wire Wire Line
+	7900 3600 8450 3600
+Wire Wire Line
+	8100 3900 8450 3900
+Wire Wire Line
+	8100 3800 8450 3800
 Wire Wire Line
 	4250 1200 4500 1200
+Wire Wire Line
+	6400 2250 6750 2250
+Wire Wire Line
+	7850 2250 7850 2450
+Connection ~ 7850 2350
+Wire Wire Line
+	6750 2350 6400 2350
+Wire Wire Line
+	6750 2450 6400 2450
+Text Label 6400 2350 0    60   ~ 0
+DI
+Text Label 6400 2450 0    60   ~ 0
+CI
+Text Label 8100 5700 0    60   ~ 0
+DI
+Text Label 8100 5800 0    60   ~ 0
+CI
+Wire Wire Line
+	8100 5800 8450 5800
+Wire Wire Line
+	8100 5700 8450 5700
 $EndSCHEMATC

Commit message: More squeezing
Parts:
- P1: footprint Pin_Headers:Pin_Header_Straight_1x02 -> Resistors_SMD:R_0805_HandSoldering
- P2: footprint Pin_Headers:Pin_Header_Straight_2x03 -> touch_timer:SIP-6-SMD
Connections:
- net 3V3: now also R4.1
Changed lines of the file:
@@
 F 0 "P2" H 5700 7500 50  0000 C CNN
 F 1 "ICSP" H 5700 7100 50  0000 C CNN
-F 2 "Pin_Headers:Pin_Header_Straight_2x03" H 5700 6100 50  0001 C CNN
+F 2 "touch_timer:SIP-6-SMD" H 5700 6100 50  0001 C CNN
 F 3 "" H 5700 6100 50  0000 C CNN
 	1    5700 7300
@@
 F 0 "P1" H 4700 1400 50  0000 C CNN
 F 1 "BATTERY" H 4950 1250 50  0000 C CNN
-F 2 "Pin_Headers:Pin_Header_Straight_1x02" H 4700 1250 50  0001 C CNN
+F 2 "Resistors_SMD:R_0805_HandSoldering" H 4700 1250 50  0001 C CNN
 F 3 "" H 4700 1250 50  0000 C CNN
 	1    4700 1250
@@
 Wire Wire Line
 	8100 5700 8450 5700
+Wire Wire Line
+	4850 4400 4850 3400
+Connection ~ 4850 3400
 $EndSCHEMATC
