File: kicad/experiments/clockface/clockface.sch (KiCad schematic (older format))
At the start: 11 parts, among them P1 BATTERY, U1 TOUCH_PAD_13, U2 MTCH6102_SSOP

Commit message: RX traces
Parts:
- removed P1: BATTERY, Resistors_SMD:R_0805_HandSoldering, symbol CONN_01X02
- added P1: CONN_01X05, Pin_Headers:Pin_Header_Straight_1x06, symbol CONN_01X05
Connections:
- net GND: now also P1.1 (P1)
- net INT: now also P1.5 (P5)
- net SCL: now also P1.4 (P4)
- net SDA: now also P1.3 (P3)
- net VCC renamed 3V3
- net 3V3: now also P1.2 (P2)
Changed lines of the file:
@@
 LIBS:contrib
 LIBS:valves
-LIBS:timer-cache
+LIBS:clockface-cache
 EELAYER 25 0
 EELAYER END
@@
 $EndComp
 $Comp
-L GND #PWR01
+L GND #PWR3
 U 1 1 57064DFC
 P 5850 3050
-F 0 "#PWR01" H 5850 2800 50  0001 C CNN
+F 0 "#PWR3" H 5850 2800 50  0001 C CNN
 F 1 "GND" H 5850 2900 50  0000 C CNN
 F 2 "" H 5850 3050 50  0000 C CNN
@@
 $EndComp
 $Comp
-L GND #PWR02
+L GND #PWR5
 U 1 1 57064DFD
 P 6350 3050
-F 0 "#PWR02" H 6350 2800 50  0001 C CNN
+F 0 "#PWR5" H 6350 2800 50  0001 C CNN
 F 1 "GND" H 6350 2900 50  0000 C CNN
 F 2 "" H 6350 3050 50  0000 C CNN
@@
 $EndComp
 $Comp
-L GND #PWR03
+L GND #PWR2
 U 1 1 57064DFE
 P 5750 5350
-F 0 "#PWR03" H 5750 5100 50  0001 C CNN
+F 0 "#PWR2" H 5750 5100 50  0001 C CNN
 F 1 "GND" H 5750 5200 50  0000 C CNN
 F 2 "" H 5750 5350 50  0000 C CNN
@@
 	1    0    0    -1
 $EndComp
-Text Label 6300 2400 0    60   ~ 0
+Text Label 6100 2200 0    60   ~ 0
 3V3
 Wire Wire Line
@@
 Connection ~ 7000 2400
 Wire Wire Line
-	6100 1800 6100 3200
+	6100 1650 6100 3200
 Connection ~ 6100 2400
 Wire Wire Line
@@
 	4400 2400 4150 2400
 $Comp
-L GND #PWR04
+L GND #PWR1
 U 1 1 57064E11
 P 3750 2550
-F 0 "#PWR04" H 3750 2300 50  0001 C CNN
+F 0 "#PWR1" H 3750 2300 50  0001 C CNN
 F 1 "GND" H 3750 2400 50  0000 C CNN
 F 2 "" H 3750 2550 50  0000 C CNN
@@
 	0    1    1    0
 $EndComp
-Wire Wire Line
-	6100 1800 6350 1800
-$Comp
-L CONN_01X02 P1
-U 1 1 57064E15
-P 6550 1850
-F 0 "P1" H 6550 2000 50  0000 C CNN
-F 1 "BATTERY" H 6800 1850 50  0000 C CNN
-F 2 "Resistors_SMD:R_0805_HandSoldering" H 6550 1850 50  0001 C CNN
-F 3 "" H 6550 1850 50  0000 C CNN
-	1    6550 1850
-	1    0    0    1
-$EndComp
-$Comp
-L GND #PWR05
+$Comp
+L GND #PWR4
 U 1 1 57064E14
-P 6350 1900
-F 0 "#PWR05" H 6350 1650 50  0001 C CNN
-F 1 "GND" H 6350 1750 50  0000 C CNN
-F 2 "" H 6350 1900 50  0000 C CNN
-F 3 "" H 6350 1900 50  0000 C CNN
-	1    6350 1900
-	1    0    0    -1
-$EndComp
-$Comp
-L VCC #PWR06
-U 1 1 57064E13
-P 6350 1800
-F 0 "#PWR06" H 6350 1650 50  0001 C CNN
-F 1 "VCC" H 6350 1950 50  0000 C CNN
-F 2 "" H 6350 1800 50  0000 C CNN
-F 3 "" H 6350 1800 50  0000 C CNN
-	1    6350 1800
+P 6000 1650
+F 0 "#PWR4" H 6000 1400 50  0001 C CNN
+F 1 "GND" H 6000 1500 50  0000 C CNN
+F 2 "" H 6000 1650 50  0000 C CNN
+F 3 "" H 6000 1650 50  0000 C CNN
+	1    6000 1650
 	1    0    0    -1
 $EndComp
@@
 Connection ~ 5750 5300
 Connection ~ 5550 5000
+$Comp
+L CONN_01X05 P1
+U 1 1 5706A4A5
+P 6200 1450
+F 0 "P1" H 6200 1750 50  0000 C CNN
+F 1 "CONN_01X05" V 6300 1450 50  0000 C CNN
+F 2 "Pin_Headers:Pin_Header_Straight_1x06" H 6200 1450 50  0001 C CNN
+F 3 "" H 6200 1450 50  0000 C CNN
+	1    6200 1450
+	0    -1   -1   0
+$EndComp
+Text Label 6200 1800 0    60   ~ 0
+SDA
+Text Label 6300 1950 0    60   ~ 0
+SCL
+Text Label 6400 2100 0    60   ~ 0
+INT
+Wire Wire Line
+	6200 1800 6200 1650
+Wire Wire Line
+	6300 1950 6300 1650
+Wire Wire Line
+	6400 2100 6400 1650
 $EndSCHEMATC

Commit message: Layed out
Parts:
- P1: footprint Pin_Headers:Pin_Header_Straight_1x06 -> clockface:SMD_Header_Straight_1x05
Connections:
- net 3V3: now also P1.1 (P1); no longer P1.2 (P2)
- net GND: now also P1.5 (P5); no longer P1.1 (P1)
- net INT: now also P1.4 (P4); no longer P1.5 (P5)
- net SCL: now also P1.2 (P2); no longer P1.4 (P4)
Changed lines of the file:
@@
 $EndComp
 $Comp
-L GND #PWR3
+L GND #PWR01
 U 1 1 57064DFC
 P 5850 3050
-F 0 "#PWR3" H 5850 2800 50  0001 C CNN
+F 0 "#PWR01" H 5850 2800 50  0001 C CNN
 F 1 "GND" H 5850 2900 50  0000 C CNN
 F 2 "" H 5850 3050 50  0000 C CNN
@@
 $EndComp
 $Comp
-L GND #PWR5
+L GND #PWR02
 U 1 1 57064DFD
 P 6350 3050
-F 0 "#PWR5" H 6350 2800 50  0001 C CNN
+F 0 "#PWR02" H 6350 2800 50  0001 C CNN
 F 1 "GND" H 6350 2900 50  0000 C CNN
 F 2 "" H 6350 3050 50  0000 C CNN
@@
 $EndComp
 $Comp
-L GND #PWR2
+L GND #PWR03
 U 1 1 57064DFE
 P 5750 5350
-F 0 "#PWR2" H 5750 5100 50  0001 C CNN
+F 0 "#PWR03" H 5750 5100 50  0001 C CNN
 F 1 "GND" H 5750 5200 50  0000 C CNN
 F 2 "" H 5750 5350 50  0000 C CNN
@@
 	1    0    0    -1
 $EndComp
-Text Label 6100 2200 0    60   ~ 0
+Text Label 6000 2250 0    60   ~ 0
 3V3
 Wire Wire Line
@@
 Connection ~ 7000 2400
 Wire Wire Line
-	6100 1650 6100 3200
-Connection ~ 6100 2400
-Wire Wire Line
 	5850 2750 6350 2750
 Connection ~ 6100 2750
@@
 	4400 2400 4150 2400
 $Comp
-L GND #PWR1
+L GND #PWR04
 U 1 1 57064E11
 P 3750 2550
-F 0 "#PWR1" H 3750 2300 50  0001 C CNN
+F 0 "#PWR04" H 3750 2300 50  0001 C CNN
 F 1 "GND" H 3750 2400 50  0000 C CNN
 F 2 "" H 3750 2550 50  0000 C CNN
@@
 $EndComp
 $Comp
-L GND #PWR4
+L GND #PWR05
 U 1 1 57064E14
-P 6000 1650
-F 0 "#PWR4" H 6000 1400 50  0001 C CNN
-F 1 "GND" H 6000 1500 50  0000 C CNN
-F 2 "" H 6000 1650 50  0000 C CNN
-F 3 "" H 6000 1650 50  0000 C CNN
-	1    6000 1650
+P 6400 1650
+F 0 "#PWR05" H 6400 1400 50  0001 C CNN
+F 1 "GND" H 6400 1500 50  0000 C CNN
+F 2 "" H 6400 1650 50  0000 C CNN
+F 3 "" H 6400 1650 50  0000 C CNN
+	1    6400 1650
 	1    0    0    -1
 $EndComp
@@
 F 0 "P1" H 6200 1750 50  0000 C CNN
 F 1 "CONN_01X05" V 6300 1450 50  0000 C CNN
-F 2 "Pin_Headers:Pin_Header_Straight_1x06" H 6200 1450 50  0001 C CNN
+F 2 "clockface:SMD_Header_Straight_1x05" H 6200 1450 50  0001 C CNN
 F 3 "" H 6200 1450 50  0000 C CNN
 	1    6200 1450
 	0    -1   -1   0
 $EndComp
-Text Label 6200 1800 0    60   ~ 0
+Text Label 6200 1950 0    60   ~ 0
 SDA
-Text Label 6300 1950 0    60   ~ 0
+Text Label 6100 1800 0    60   ~ 0
 SCL
-Text Label 6400 2100 0    60   ~ 0
+Text Label 6300 2100 0    60   ~ 0
 INT
 Wire Wire Line
-	6200 1800 6200 1650
+	6200 1650 6200 1950
 Wire Wire Line
-	6300 1950 6300 1650
+	6300 1650 6300 2100
 Wire Wire Line
-	6400 2100 6400 1650
+	6000 1650 6000 2600
+Connection ~ 6000 2400
+Wire Wire Line
+	6100 1650 6100 1800
+Wire Wire Line
+	6100 2600 6100 3200
+Wire Wire Line
+	6000 2600 6100 2600
+$Comp
+L GND #PWR?
+U 1 1 5706D7C6
+P 3700 3600
+F 0 "#PWR?" H 3700 3350 50  0001 C CNN
+F 1 "GND" H 3700 3450 50  0000 C CNN
+F 2 "" H 3700 3600 50  0000 C CNN
+F 3 "" H 3700 3600 50  0000 C CNN
+	1    3700 3600
+	1    0    0    -1
+$EndComp
 $EndSCHEMATC

Commit message: Soldermask on the ic footprint
Parts:
- U2: footprint Housings_SSOP:SSOP-28_5.3x10.2mm_Pitch0.65mm -> clockface:SSOP-28_5.3x10.2mm_Pitch0.65mm_masked
Changed lines of the file:
@@
 F 0 "U2" H 6300 3300 60  0000 C CNN
 F 1 "MTCH6102_SSOP" H 6800 1350 60  0000 C CNN
-F 2 "Housings_SSOP:SSOP-28_5.3x10.2mm_Pitch0.65mm" H 6100 3300 60  0001 C CNN
+F 2 "clockface:SSOP-28_5.3x10.2mm_Pitch0.65mm_masked" H 6100 3300 60  0001 C CNN
 F 3 "" H 6100 3300 60  0000 C CNN
 	1    6100 3300
