File: kicad/ada/timer.sch (KiCad schematic (older format))
At the start: 27 parts, among them IC1 ATMEGA328P-A, P1 BATTERY, P2 ICSP, Q1 NMOS, Q2 PMOS, SW1 SPST, U1 TOUCH_PAD_13, U2 MTCH6102_SSOP, U3 MCP1755ST-3302E/DB, U4 APA_102C

Commit message: Start of using clockface
Parts:
- removed R5: 4.7k, Resistors_SMD:R_0805_HandSoldering, symbol R
- U1: footprint touch_timer:touch_circle -> touch_timer:CPA_12
- U2: footprint Housings_SSOP:SSOP-28_5.3x10.2mm_Pitch0.65mm -> touch_timer:SSOP-28_5.3x10.2mm_Pitch0.65mm_masked
Connections:
- net 3V3: now also U4.4 (VCC)
- net GND: now also U1.14 (GND)
- net POWER: no longer U4.4 (VCC)
- net SYNC: no longer names the net of U2.12 (SYNC)
Changed lines of the file:
@@
 LIBS:valves
 LIBS:timer-cache
-LIBS:rc_power_sockets-cache
 EELAYER 25 0
 EELAYER END
@@
 F 0 "U2" H 3750 4300 60  0000 C CNN
 F 1 "MTCH6102_SSOP" H 4250 2350 60  0000 C CNN
-F 2 "Housings_SSOP:SSOP-28_5.3x10.2mm_Pitch0.65mm" H 3550 4300 60  0001 C CNN
+F 2 "touch_timer:SSOP-28_5.3x10.2mm_Pitch0.65mm_masked" H 3550 4300 60  0001 C CNN
 F 3 "" H 3550 4300 60  0000 C CNN
 	1    3550 4300
@@
 F 0 "U1" H 1700 2650 60  0000 C CNN
 F 1 "TOUCH_PAD_13" H 1700 4500 60  0000 C CNN
-F 2 "touch_timer:touch_circle" H 1700 4400 60  0001 C CNN
+F 2 "touch_timer:CPA_12" H 1700 4400 60  0001 C CNN
 F 3 "" H 1700 4400 60  0000 C CNN
 	1    1700 4400
@@
 	1    0    0    -1
 $EndComp
-$Comp
-L R R5
-U 1 1 5704F67F
-P 5050 4650
-F 0 "R5" V 5130 4650 50  0000 C CNN
-F 1 "4.7k" V 5050 4650 50  0000 C CNN
-F 2 "Resistors_SMD:R_0805_HandSoldering" V 4980 4650 50  0001 C CNN
-F 3 "" H 5050 4650 50  0000 C CNN
-	1    5050 4650
-	1    0    0    -1
-$EndComp
-Text Label 4150 4800 0    60   ~ 0
-SYNC
 $Comp
 L R R1
@@
 $EndComp
 $Comp
-L VCC #PWR010
-U 1 1 57056634
-P 4500 1200
-F 0 "#PWR010" H 4500 1050 50  0001 C CNN
-F 1 "VCC" H 4500 1350 50  0000 C CNN
-F 2 "" H 4500 1200 50  0000 C CNN
-F 3 "" H 4500 1200 50  0000 C CNN
-	1    4500 1200
-	1    0    0    -1
-$EndComp
-$Comp
-L GND #PWR011
+L GND #PWR010
 U 1 1 57056635
 P 4500 1300
-F 0 "#PWR011" H 4500 1050 50  0001 C CNN
+F 0 "#PWR010" H 4500 1050 50  0001 C CNN
 F 1 "GND" H 4500 1150 50  0000 C CNN
 F 2 "" H 4500 1300 50  0000 C CNN
@@
 $EndComp
 $Comp
-L GND #PWR012
+L GND #PWR011
 U 1 1 57057D8A
 P 7800 5250
-F 0 "#PWR012" H 7800 5000 50  0001 C CNN
+F 0 "#PWR011" H 7800 5000 50  0001 C CNN
 F 1 "GND" H 7800 5100 50  0000 C CNN
 F 2 "" H 7800 5250 50  0000 C CNN
@@
 	1    0    0    -1
 $EndComp
-Text Label 6400 2250 0    60   ~ 0
-POWER
-$Comp
-L GND #PWR013
+$Comp
+L GND #PWR012
 U 1 1 570638A5
 P 7850 2450
-F 0 "#PWR013" H 7850 2200 50  0001 C CNN
+F 0 "#PWR012" H 7850 2200 50  0001 C CNN
 F 1 "GND" H 7850 2300 50  0000 C CNN
 F 2 "" H 7850 2450 50  0000 C CNN
@@
 	2250 5800 3000 5800
 Wire Wire Line
-	4100 4800 5050 4800
-Wire Wire Line
 	4450 3400 4450 4200
 Wire Wire Line
-	2550 3400 5050 3400
+	2550 3400 4850 3400
 Wire Wire Line
 	4650 4300 4650 3400
 Connection ~ 4650 3400
-Wire Wire Line
-	5050 3400 5050 4500
 Wire Wire Line
 	3000 4500 2550 4500
@@
 	8100 5700 8450 5700
 Wire Wire Line
-	4850 4400 4850 3400
+	4850 3400 4850 4400
 Connection ~ 4850 3400
+Text Label 4250 1200 0    60   ~ 0
+VCC
+Text Label 6400 2250 0    60   ~ 0
+3V3
+$Comp
+L GND #PWR013
+U 1 1 570E41B7
+P 1150 4600
+F 0 "#PWR013" H 1150 4350 50  0001 C CNN
+F 1 "GND" H 1150 4450 50  0000 C CNN
+F 2 "" H 1150 4600 50  0000 C CNN
+F 3 "" H 1150 4600 50  0000 C CNN
+	1    1150 4600
+	1    0    0    -1
+$EndComp
 $EndSCHEMATC
