File: kicad/experiments/atmega/atmega.sch (KiCad schematic (older format))
At the start: 8 parts, among them IC1 ATMEGA328P-A, P1 ISCP, P2 SERIAL, P3 CONN_01X05

Commit message: Layout
Parts:
- removed P2: SERIAL, Pin_Headers:Pin_Header_Straight_1x03, symbol CONN_01X03
- added C3: 0.1uF, Capacitors_SMD:C_0805_HandSoldering, symbol C
- added P2: FTDI, Socket_Strips:Socket_Strip_Straight_1x06, symbol CONN_01X06
- added P4: GPIO, theapi:SMD_Header_Straight_1x05, symbol CONN_01X05
- added R2: 10k, Resistors_SMD:R_0805_HandSoldering, symbol R
- P3: value CONN_01X05 -> I2C; footprint Pin_Headers:Pin_Header_Straight_1x05 -> theapi:SMD_Header_Straight_1x05
Connections:
- net CLK is gone; now on net SCK: P1.3 (P3)
- net +3V3: now also P2.3 (P3), R2.1
- net GND: now also P2.1 (P1), P2.2 (P2)
- net PB1: now also P4.1 (P1)
- net PB2/SS: now also P4.2 (P2)
- net PD3: now also P4.5 (P5)
- net PD5: now also P4.3 (P3)
- net PD6: now also P4.4 (P4)
- net RESET: now also C3.2, R2.2
- net RX: now also P2.5 (P5)
- net TX: now also P2.4 (P4)
- new net DTR: C3.1, P2.6 (P6)
Other:
- moved on the sheet: P3
Changed lines of the file:
@@
 LIBS:contrib
 LIBS:valves
+LIBS:atmega-cache
 EELAYER 25 0
 EELAYER END
@@
 	6700 3750 6900 3750
 Wire Wire Line
-	6700 3850 6900 3850
+	6700 3850 7500 3850
 Text Label 4300 2250 0    60   ~ 0
 3V3
@@
 MISO
 Text Label 8600 1650 0    60   ~ 0
-CLK
+SCK
 Text Label 8600 1750 0    60   ~ 0
 RESET
@@
 	9400 1650 9550 1650
 $Comp
-L CONN_01X03 P2
-U 1 1 5730C01F
-P 9150 2600
-F 0 "P2" H 9150 2800 50  0000 C CNN
-F 1 "SERIAL" V 9250 2600 50  0000 C CNN
-F 2 "Pin_Headers:Pin_Header_Straight_1x03" H 9150 2600 50  0001 C CNN
-F 3 "" H 9150 2600 50  0000 C CNN
-	1    9150 2600
-	1    0    0    1
-$EndComp
-$Comp
 L GND #PWR05
-U 1 1 5730C07A
-P 8950 2700
-F 0 "#PWR05" H 8950 2450 50  0001 C CNN
-F 1 "GND" H 8950 2550 50  0000 C CNN
-F 2 "" H 8950 2700 50  0000 C CNN
-F 3 "" H 8950 2700 50  0000 C CNN
-	1    8950 2700
-	1    0    0    -1
-$EndComp
-Text Label 8700 2500 0    60   ~ 0
-RX
-Text Label 8700 2600 0    60   ~ 0
-TX
-Wire Wire Line
-	8700 2600 8950 2600
-Wire Wire Line
-	8700 2500 8950 2500
-$Comp
-L GND #PWR06
 U 1 1 5730C1EC
-P 8950 4250
-F 0 "#PWR06" H 8950 4000 50  0001 C CNN
-F 1 "GND" H 8950 4100 50  0000 C CNN
-F 2 "" H 8950 4250 50  0000 C CNN
-F 3 "" H 8950 4250 50  0000 C CNN
-	1    8950 4250
-	1    0    0    -1
-$EndComp
-Text Label 8700 3950 0    60   ~ 0
+P 9300 4000
+F 0 "#PWR05" H 9300 3750 50  0001 C CNN
+F 1 "GND" H 9300 3850 50  0000 C CNN
+F 2 "" H 9300 4000 50  0000 C CNN
+F 3 "" H 9300 4000 50  0000 C CNN
+	1    9300 4000
+	1    0    0    -1
+$EndComp
+Text Label 9050 3700 0    60   ~ 0
 SDA
-Text Label 8700 4050 0    60   ~ 0
+Text Label 9050 3800 0    60   ~ 0
 SCL
 Wire Wire Line
-	8700 3950 8950 3950
-Wire Wire Line
-	8700 4050 8950 4050
+	9050 3700 9300 3700
+Wire Wire Line
+	9050 3800 9300 3800
 $Comp
 L CONN_01X05 P3
 U 1 1 5730C351
-P 9150 4050
-F 0 "P3" H 9150 4350 50  0000 C CNN
-F 1 "CONN_01X05" V 9250 4050 50  0000 C CNN
-F 2 "Pin_Headers:Pin_Header_Straight_1x05" H 9150 4050 50  0001 C CNN
-F 3 "" H 9150 4050 50  0000 C CNN
-	1    9150 4050
+P 9500 3800
+F 0 "P3" H 9500 4100 50  0000 C CNN
+F 1 "I2C" V 9600 3800 50  0000 C CNN
+F 2 "theapi:SMD_Header_Straight_1x05" H 9500 3800 50  0001 C CNN
+F 3 "" H 9500 3800 50  0000 C CNN
+	1    9500 3800
 	1    0    0    1
 $EndComp
-Text Label 8700 3850 0    60   ~ 0
+Text Label 9050 3600 0    60   ~ 0
 INT0
-Text Label 8700 4150 0    60   ~ 0
-3V3
-Wire Wire Line
-	8700 4150 8950 4150
-Wire Wire Line
-	8700 3850 8950 3850
+Wire Wire Line
+	8850 3900 9300 3900
+Wire Wire Line
+	9050 3600 9300 3600
 $Comp
 L C C2
@@
 Connection ~ 3850 2400
 $Comp
-L GND #PWR07
+L GND #PWR06
 U 1 1 5730C767
 P 3400 2700
-F 0 "#PWR07" H 3400 2450 50  0001 C CNN
+F 0 "#PWR06" H 3400 2450 50  0001 C CNN
 F 1 "GND" H 3400 2550 50  0000 C CNN
 F 2 "" H 3400 2700 50  0000 C CNN
@@
 $EndComp
 $Comp
-L GND #PWR08
+L GND #PWR07
 U 1 1 5730C7CA
 P 6200 1650
-F 0 "#PWR08" H 6200 1400 50  0001 C CNN
+F 0 "#PWR07" H 6200 1400 50  0001 C CNN
 F 1 "GND" H 6200 1500 50  0000 C CNN
 F 2 "" H 6200 1650 50  0000 C CNN
@@
 NoConn ~ 6700 4400
 NoConn ~ 6700 4700
+$Comp
+L R R2
+U 1 1 5730E2EA
+P 7500 3700
+F 0 "R2" V 7580 3700 50  0000 C CNN
+F 1 "10k" V 7500 3700 50  0000 C CNN
+F 2 "Resistors_SMD:R_0805_HandSoldering" V 7430 3700 50  0001 C CNN
+F 3 "" H 7500 3700 50  0000 C CNN
+	1    7500 3700
+	1    0    0    -1
+$EndComp
+$Comp
+L +3.3V #PWR08
+U 1 1 5730E31C
+P 7500 3550
+F 0 "#PWR08" H 7500 3400 50  0001 C CNN
+F 1 "+3.3V" H 7500 3690 50  0000 C CNN
+F 2 "" H 7500 3550 50  0000 C CNN
+F 3 "" H 7500 3550 50  0000 C CNN
+	1    7500 3550
+	1    0    0    -1
+$EndComp
+$Comp
+L CONN_01X06 P2
+U 1 1 5730E4F7
+P 9500 2750
+F 0 "P2" H 9500 3100 50  0000 C CNN
+F 1 "FTDI" V 9600 2750 50  0000 C CNN
+F 2 "Socket_Strips:Socket_Strip_Straight_1x06" H 9500 2750 50  0001 C CNN
+F 3 "" H 9500 2750 50  0000 C CNN
+	1    9500 2750
+	1    0    0    -1
+$EndComp
+$Comp
+L GND #PWR09
+U 1 1 5730E695
+P 8750 2600
+F 0 "#PWR09" H 8750 2350 50  0001 C CNN
+F 1 "GND" H 8750 2450 50  0000 C CNN
+F 2 "" H 8750 2600 50  0000 C CNN
+F 3 "" H 8750 2600 50  0000 C CNN
+	1    8750 2600
+	1    0    0    -1
+$EndComp
+Text Label 9050 2900 0    60   ~ 0
+RX
+Text Label 9050 2800 0    60   ~ 0
+TX
+$Comp
+L +3.3V #PWR010
+U 1 1 5730E6FE
+P 9000 2700
+F 0 "#PWR010" H 9000 2550 50  0001 C CNN
+F 1 "+3.3V" H 9000 2840 50  0000 C CNN
+F 2 "" H 9000 2700 50  0000 C CNN
+F 3 "" H 9000 2700 50  0000 C CNN
+	1    9000 2700
+	1    0    0    -1
+$EndComp
+Text Label 9050 3000 0    60   ~ 0
+DTR
+Wire Wire Line
+	9050 3000 9300 3000
+Wire Wire Line
+	9300 2900 9050 2900
+Wire Wire Line
+	9050 2800 9300 2800
+Wire Wire Line
+	9300 2700 9000 2700
+Wire Wire Line
+	9300 2500 9300 2600
+Wire Wire Line
+	8750 2500 9300 2500
+Wire Wire Line
+	8750 2500 8750 2600
+Text Label 9050 4700 0    60   ~ 0
+PB1
+Text Label 8900 4800 0    60   ~ 0
+PB2/SS
+Text Label 9050 5100 0    60   ~ 0
+PD3
+Text Label 9050 4900 0    60   ~ 0
+PD5
+Text Label 9050 5000 0    60   ~ 0
+PD6
+$Comp
+L CONN_01X05 P4
+U 1 1 5730ECDF
+P 9500 4900
+F 0 "P4" H 9500 5200 50  0000 C CNN
+F 1 "GPIO" V 9600 4900 50  0000 C CNN
+F 2 "theapi:SMD_Header_Straight_1x05" H 9500 4900 50  0001 C CNN
+F 3 "" H 9500 4900 50  0000 C CNN
+	1    9500 4900
+	1    0    0    -1
+$EndComp
+Wire Wire Line
+	9050 4700 9300 4700
+Wire Wire Line
+	9300 4800 8900 4800
+Wire Wire Line
+	9300 4900 9050 4900
+Wire Wire Line
+	9300 5000 9050 5000
+Wire Wire Line
+	9300 5100 9050 5100
+$Comp
+L C C3
+U 1 1 5730F2C0
+P 7650 3850
+F 0 "C3" H 7675 3950 50  0000 L CNN
+F 1 "0.1uF" H 7675 3750 50  0000 L CNN
+F 2 "Capacitors_SMD:C_0805_HandSoldering" H 7688 3700 50  0001 C CNN
+F 3 "" H 7650 3850 50  0000 C CNN
+	1    7650 3850
+	0    1    1    0
+$EndComp
+Text Label 7950 3850 0    60   ~ 0
+DTR
+Wire Wire Line
+	7800 3850 7950 3850
+$Comp
+L +3.3V #PWR011
+U 1 1 5730F4E6
+P 8850 3900
+F 0 "#PWR011" H 8850 3750 50  0001 C CNN
+F 1 "+3.3V" H 8850 4040 50  0000 C CNN
+F 2 "" H 8850 3900 50  0000 C CNN
+F 3 "" H 8850 3900 50  0000 C CNN
+	1    8850 3900
+	1    0    0    -1
+$EndComp
 $EndSCHEMATC

Commit message: Through hole headers
Parts:
- P3, P4: footprint theapi:SMD_Header_Straight_1x05 -> Pin_Headers:Pin_Header_Straight_1x05
Connections:
- net PB1: now also P4.2 (P2); no longer P4.1 (P1)
- net PB2/SS: now also P4.1 (P1); no longer P4.2 (P2)
- net PD5: now also P4.4 (P4); no longer P4.3 (P3)
- net PD6: now also P4.3 (P3); no longer P4.4 (P4)
- net RX: now also P2.4 (P4); no longer P2.5 (P5)
- net SCL: now also P3.4 (P4); no longer P3.3 (P3)
- net SDA: now also P3.3 (P3); no longer P3.4 (P4)
- net TX: now also P2.5 (P5); no longer P2.4 (P4)
Changed lines of the file:
@@
 	1    0    0    -1
 $EndComp
+Text Label 9050 3800 0    60   ~ 0
+SDA
 Text Label 9050 3700 0    60   ~ 0
-SDA
-Text Label 9050 3800 0    60   ~ 0
 SCL
 Wire Wire Line
@@
 F 0 "P3" H 9500 4100 50  0000 C CNN
 F 1 "I2C" V 9600 3800 50  0000 C CNN
-F 2 "theapi:SMD_Header_Straight_1x05" H 9500 3800 50  0001 C CNN
+F 2 "Pin_Headers:Pin_Header_Straight_1x05" H 9500 3800 50  0001 C CNN
 F 3 "" H 9500 3800 50  0000 C CNN
 	1    9500 3800
@@
 	1    0    0    -1
 $EndComp
+Text Label 9050 2800 0    60   ~ 0
+RX
 Text Label 9050 2900 0    60   ~ 0
-RX
-Text Label 9050 2800 0    60   ~ 0
 TX
 $Comp
@@
 Wire Wire Line
 	8750 2500 8750 2600
-Text Label 9050 4700 0    60   ~ 0
+Text Label 9050 4800 0    60   ~ 0
 PB1
-Text Label 8900 4800 0    60   ~ 0
+Text Label 8900 4700 0    60   ~ 0
 PB2/SS
 Text Label 9050 5100 0    60   ~ 0
 PD3
+Text Label 9050 5000 0    60   ~ 0
+PD5
 Text Label 9050 4900 0    60   ~ 0
-PD5
-Text Label 9050 5000 0    60   ~ 0
 PD6
 $Comp
@@
 F 0 "P4" H 9500 5200 50  0000 C CNN
 F 1 "GPIO" V 9600 4900 50  0000 C CNN
-F 2 "theapi:SMD_Header_Straight_1x05" H 9500 4900 50  0001 C CNN
+F 2 "Pin_Headers:Pin_Header_Straight_1x05" H 9500 4900 50  0001 C CNN
 F 3 "" H 9500 4900 50  0000 C CNN
 	1    9500 4900
@@
 $EndComp
 Wire Wire Line
-	9050 4700 9300 4700
+	8900 4700 9300 4700
 Wire Wire Line
-	9300 4800 8900 4800
+	9300 4800 9050 4800
 Wire Wire Line
 	9300 4900 9050 4900
